Commit message: latest

File: rrbot_description/urdf/rrbot.xacro (robot description, xacro)
@@ -1,14 +1,53 @@
 <?xml version="1.0"?>
-<!-- Revolute-Revolute Manipulator -->
 <robot name="rrbot" xmlns:xacro="http://www.ros.org/wiki/xacro">
   <!-- Constants for robot dimensions -->
   <xacro:property name="PI" value="3.1415926535897931"/>
-  <xacro:property name="mass" value="1" /> <!-- arbitrary value for mass -->
-  <xacro:property name="width" value="0.1" /> <!-- Square dimensions (widthxwidth) of beams -->
-  <xacro:property name="height1" value="2" /> <!-- Link 1 -->
-  <xacro:property name="height2" value="1" /> <!-- Link 2 -->
-  <xacro:property name="height3" value="1" /> <!-- Link 3 -->
-  <xacro:property name="camera_link" value="0.05" /> <!-- Size of square 'camera' box -->
-  <xacro:property name="axel_offset" value="0.05" /> <!-- Space btw top of beam and the each joint -->
+  <xacro:property name="mass" value="2.0" /> <!-- arbitrary value for mass -->
+  <xacro:property name="width" value="0.05" /> <!-- Square dimensions (widthxwidth) of beams -->
+  <xacro:property name="ry" value="0.016" />
+  <xacro:property name="rz" value="0.02" />
+  <xacro:property name="height1" value="1.5" /> <!-- Link 1 -->
+  <xacro:property name="height2" value="0.25" /> <!-- Link 2 -->
+  <xacro:property name="height3" value="0.4" /> <!-- Link 3 -->
+  <xacro:property name="height4" value="0.4" /><!-- Link4 -->
+  <xacro:property name="height_w1" value="0.03" />
+  <xacro:property name="width_w1" value="0.02" />
+  <xacro:property name="mass_w1" value="1" />
+  <xacro:property name="height_w2" value="0.03" />
+  <xacro:property name="width_w2" value="0.02" />
+  <xacro:property name="mass_w2" value="1" />
+  <xacro:property name="height_p" value="0.1" />
+  <xacro:property name="width_p" value="0.09" />
+  <xacro:property name="mass_p" value="1" />
+  <xacro:property name="height_t" value="0.03" />
+  <xacro:property name="width_t" value="0.02" />
+  <xacro:property name="mass_t" value="1" />
+  <xacro:property name="height_i" value="0.03" />
+  <xacro:property name="width_i" value="0.02" />
+  <xacro:property name="mass_i" value="1" />
+  <xacro:property name="height_m" value="0.03" />
+  <xacro:property name="width_m" value="0.02" />
+  <xacro:property name="mass_m" value="1" />
+  <xacro:property name="height_s" value="0.03" />
+  <xacro:property name="width_s" value="0.02" />
+  <xacro:property name="mass_s" value="1" />
+  <xacro:property name="height_l" value="0.03" />
+  <xacro:property name="width_l" value="0.02" />
+  <xacro:property name="mass_l" value="1" />
+  <xacro:property name="rl" value="${sqrt((rz+height4)*(rz+height4)+ry*ry)}" />
+  <xacro:property name="model_scale" value="0.6 0.6 0.6" />
+  <xacro:property name="model_humerus" value="package://rrbot_description/meshes/humerus_0.1_r.dae" />
+  <xacro:property name="model_radius" value="package://rrbot_description/meshes/radius_0.1_t.dae" />
+  <xacro:property name="model_ulna" value="package://rrbot_description/meshes/ulna_0.1_r.dae" />
+  <xacro:property name="model_hand" value="package://rrbot_description/meshes/hand.dae" />
+  <xacro:property name="model_wrist1" value="package://rrbot_description/meshes/hand/wrist1.dae" />
+  <xacro:property name="model_wrist2" value="package://rrbot_description/meshes/hand/wrist2.dae" />
+  <xacro:property name="model_palm" value="package://rrbot_description/meshes/hand/palm.dae" />
+<xacro:property name="model_thumb1" value="package://rrbot_description/meshes/hand/thumb1.dae" />
+<xacro:property name="model_thumb2" value="package://rrbot_description/meshes/hand/thumb2.dae" />
+<xacro:property name="model_thumb3" value="package://rrbot_description/meshes/hand/thumb3.dae" />
+<xacro:property name="model_index1" value="package://rrbot_description/meshes/hand/index1.dae" />
+<xacro:property name="model_index2" value="package://rrbot_description/meshes/hand/index2.dae" />
+<xacro:property name="model_index3" value="package://rrbot_description/meshes/hand/index3.dae" />
   <!-- Import all Gazebo-customization elements, including Gazebo colors -->
   <xacro:include filename="$(find rrbot_description)/urdf/rrbot.gazebo" />
@@ -40,13 +79,43 @@
       <mass value="${mass}"/>
       <inertia
-	  ixx="${mass / 12.0 * (width*width + height1*height1)}" ixy="0.0" ixz="0.0"
-	  iyy="${mass / 12.0 * (height1*height1 + width*width)}" iyz="0.0"
-	  izz="${mass / 12.0 * (width*width + width*width)}"/>
-    </inertial>
-  </link>
-  <joint name="joint1" type="continuous">
+	  ixx="${mass / 1.0  * (width*width + height1*height1)}" ixy="0.0" ixz="0.0"
+	  iyy="${mass / 1.0  * (height1*height1 + width*width)}" iyz="0.0"
+	  izz="${mass / 1.0  * (width*width + width*width)}"/>
+    </inertial>
+  </link>
+  <joint name="joint_bridge" type="fixed">
     <parent link="link1"/>
+    <child link="link_bridge"/>
+	<origin xyz="0 ${width} ${height1 - width/2}" rpy="0 0 0"/>
+    <axis xyz="0 1 0"/>
+    <dynamics damping="0.7"/>
+  </joint>
+  <link name="link_bridge">
+    <collision>
+		<origin xyz="0 ${width*3/2} 0" rpy="0 0 0"/>
+      <geometry>
+	<box size="${width} ${width*3} ${width}"/>
+      </geometry>
+    </collision>
+    <visual>
+		<origin xyz="0 ${width} 0" rpy="0 0 0"/>
+      <geometry>
+	<box size="${width} ${width*3} ${width}"/>
+      </geometry>
+      <material name="orange"/>
+    </visual>
+    <inertial>
+		<origin xyz="0 ${width} 0" rpy="0 0 0"/>
+      <mass value="${mass}"/>
+      <inertia
+	  ixx="${mass / 1.0  * (width*width + width*width)}" ixy="0.0" ixz="0.0"
+	  iyy="${mass / 1.0  * (width*width + width*width)}" iyz="0.0"
+	  izz="${mass / 1.0  * (width*width + width*width)}"/>
+    </inertial>
+  </link>
+  <joint name="joint1" type="fixed">
+    <parent link="link_bridge"/>
     <child link="link2"/>
-    <origin xyz="0 ${width} ${height1 - axel_offset}" rpy="0 0 0"/>
+	<origin xyz="0 ${width*3} -0.05" rpy="0 ${PI} 0"/>
     <axis xyz="0 1 0"/>
     <dynamics damping="0.7"/>
@@ -55,23 +124,25 @@
   <link name="link2">
     <collision>
-      <origin xyz="0 0 ${height2/2 - axel_offset}" rpy="0 0 0"/>
-      <geometry>
-	<box size="${width} ${width} ${height2}"/>
-      </geometry>
-    </collision>
-    <visual>
-      <origin xyz="0 0 ${height2/2 - axel_offset}" rpy="0 0 0"/>
-      <geometry>
-	<box size="${width} ${width} ${height2}"/>
-      </geometry>
-      <material name="black"/>
-    </visual>
-    <inertial>
-      <origin xyz="0 0 ${height2/2 - axel_offset}" rpy="0 0 0"/>
+      <origin xyz="0 0 ${height2/2}" rpy="0 0 0"/>
+      <geometry>
+	<!--box size="${width} ${width} ${height2}"/-->
+	<mesh filename="${model_humerus}" scale="${model_scale}" />
+      </geometry>
+    </collision>
+    <visual>
+      <origin xyz="0 0 ${height2/2}" rpy="0 0 0"/>
+      <geometry>
+		  <!--box size="${width} ${width} ${height2}"/-->
+		<mesh filename="${model_humerus}" scale="${model_scale}" />
+      </geometry>
+      <!--material name="black"/-->
+    </visual>
+    <inertial>
+      <origin xyz="0 0 ${height2/2}" rpy="0 0 0"/>
       <mass value="${mass}"/>
       <inertia
-	  ixx="${mass / 12.0 * (width*width + height2*height2)}" ixy="0.0" ixz="0.0"
-	  iyy="${mass / 12.0 * (height2*height2 + width*width)}" iyz="0.0"
-	  izz="${mass / 12.0 * (width*width + width*width)}"/>
+	  ixx="${mass / 1.0  * (width*width + height2*height2)}" ixy="0.0" ixz="0.0"
+	  iyy="${mass / 1.0  * (height2*height2 + width*width)}" iyz="0.0"
+	  izz="${mass / 1.0  * (width*width + width*width)}"/>
     </inertial>
   </link>
@@ -79,96 +150,633 @@
     <parent link="link2"/>
     <child link="link3"/>
-    <origin xyz="0 ${width} ${height2 - axel_offset*2}" rpy="0 0 0"/>
-    <axis xyz="0 1 0"/>
-    <dynamics damping="0.7"/>
-  </joint>
-  <!-- Top Link -->
+	<origin xyz="0.04 0 ${height2}" rpy="0 0 0"/>
+	<axis xyz="0 1 0"/>
+    <dynamics damping="0.7"/>
+  </joint>
   <link name="link3">
     <collision>
-      <origin xyz="0 0 ${height3/2 - axel_offset}" rpy="0 0 0"/>
-      <geometry>
-	<box size="${width} ${width} ${height3}"/>
-      </geometry>
-    </collision>
-    <visual>
-      <origin xyz="0 0 ${height3/2 - axel_offset}" rpy="0 0 0"/>
-      <geometry>
-	<box size="${width} ${width} ${height3}"/>
-      </geometry>
-      <material name="orange"/>
-    </visual>
-    <inertial>
-      <origin xyz="0 0 ${height3/2 - axel_offset}" rpy="0 0 0"/>
+		<origin xyz="0 0 ${height3/2}" rpy="0 0 0"/>
+      <geometry>
+		  <!--box size="${width} ${width} ${height3}"/-->
+		<mesh filename="${model_ulna}" scale="${model_scale}" />
+      </geometry>
+    </collision>
+    <visual>
+		<origin xyz="0 0 ${height3/2}" rpy="0 0 0"/>
+      <geometry>
+	<!--box size="${width} ${width} ${height3}"/-->
+	<mesh filename="${model_ulna}" scale="${model_scale}" />
+      </geometry>
+      <material name="orange"/>
+    </visual>
+    <inertial>
+		<origin xyz="0 0 ${height3/2}" rpy="0 0 0"/>
       <mass value="${mass}"/>
       <inertia
-	  ixx="${mass / 12.0 * (width*width + height3*height3)}" ixy="0.0" ixz="0.0"
-	  iyy="${mass / 12.0 * (height3*height3 + width*width)}" iyz="0.0"
-	  izz="${mass / 12.0 * (width*width + width*width)}"/>
-    </inertial>
-  </link>
-  <joint name="hokuyo_joint" type="fixed">
-    <axis xyz="0 1 0" />
-    <origin xyz="0 0 ${height3 - axel_offset/2}" rpy="0 0 0"/>
+	  ixx="${mass / 1.0  * (width*width + height3*height3)}" ixy="0.0" ixz="0.0"
+	  iyy="${mass / 1.0  * (height3*height3 + width*width)}" iyz="0.0"
+	  izz="${mass / 1.0  * (width*width + width*width)}"/>
+    </inertial>
+  </link>
+  <joint name="joint3" type="continuous">
     <parent link="link3"/>
-    <child link="hokuyo_link"/>
-  </joint>
-  <!-- Hokuyo Laser -->
-  <link name="hokuyo_link">
-    <collision>
-      <origin xyz="0 0 0" rpy="0 0 0"/>
-      <geometry>
-	<box size="0.1 0.1 0.1"/>
-      </geometry>
-    </collision>
-    <visual>
-      <origin xyz="0 0 0" rpy="0 0 0"/>
-      <geometry>
-        <mesh filename="package://rrbot_description/meshes/hokuyo.dae"/>
-      </geometry>
-    </visual>
-    <inertial>
-      <mass value="1e-5" />
-      <origin xyz="0 0 0" rpy="0 0 0"/>
-      <inertia ixx="1e-6" ixy="0" ixz="0" iyy="1e-6" iyz="0" izz="1e-6" />
-    </inertial>
-  </link>
-  <joint name="camera_joint" type="fixed">
-    <axis xyz="0 1 0" />
-    <origin xyz="${camera_link} 0 ${height3 - axel_offset*2}" rpy="0 0 0"/>
-    <parent link="link3"/>
-    <child link="camera_link"/>
-  </joint>
-  <!-- Camera -->
-  <link name="camera_link">
-    <collision>
-      <origin xyz="0 0 0" rpy="0 0 0"/>
-      <geometry>
-	<box size="${camera_link} ${camera_link} ${camera_link}"/>
-      </geometry>
-    </collision>
-    <visual>
-      <origin xyz="0 0 0" rpy="0 0 0"/>
-      <geometry>
-	<box size="${camera_link} ${camera_link} ${camera_link}"/>
-      </geometry>
-      <material name="red"/>
-    </visual>
-    <inertial>
-      <mass value="1e-5" />
-      <origin xyz="0 0 0" rpy="0 0 0"/>
-      <inertia ixx="1e-6" ixy="0" ixz="0" iyy="1e-6" iyz="0" izz="1e-6" />
-    </inertial>
-  </link>
-  <!-- generate an optical frame http://www.ros.org/reps/rep-0103.html#suffix-frames
-      so that ros and opencv can operate on the camera frame correctly -->
-  <joint name="camera_optical_joint" type="fixed">
-    <!-- these values have to be these values otherwise the gazebo camera image
-        won't be aligned properly with the frame it is supposedly originating from -->
-    <origin xyz="0 0 0" rpy="${-pi/2} 0 ${-pi/2}"/>
-    <parent link="camera_link"/>
-    <child link="camera_link_optical"/>
-  </joint>
-  <link name="camera_link_optical">
-  </link>
+    <child link="link4"/>
+	<origin xyz="-0.014 ${ry} ${rz}" rpy="0 0 0"/>
+	<axis xyz="0 ${-ry/rl} ${(rz+height4)/rl}"/>
+	<!--axis xyz="0 0 1" /-->
+    <dynamics damping="0.7"/>
+  </joint>
+  <link name="link4">
+    <collision>
+		<origin xyz="0 0 ${height4/2}" rpy="0 0 0"/>
+      <geometry>
+		  <!--box size="${width} ${width} ${height4}"/-->
+     	<mesh filename="${model_radius}" scale="${model_scale}" />
+      </geometry>
+    </collision>
+    <visual>
+		<origin xyz="0 0 ${height4/2}" rpy="0 0 0"/>
+      <geometry>
+		<!--box size="${width} ${width} ${height4}"/-->
+		<mesh filename="${model_radius}" scale="${model_scale}" />
+      </geometry>
+      <material name="orange"/>
+    </visual>
+    <inertial>
+		<origin xyz="0 0 ${height4/2}" rpy="0 0 0"/>
+      <mass value="${mass}"/>
+      <inertia
+	  ixx="${mass / 1.0  * (width*width + height4*height4)}" ixy="0.0" ixz="0.0"
+	  iyy="${mass / 1.0  * (height4*height4 + width*width)}" iyz="0.0"
+	  izz="${mass / 1.0  * (width*width + width*width)}"/>
+    </inertial>
+  </link>
+<!--********************* WRIST *********************** -->
+  <joint name="wrist_joint1" type="continuous">
+    <parent link="link4"/>
+    <child link="wrist_link1"/>
+		<origin xyz="-0.0025 0 ${height4-0.01}" rpy="0 0 0"/>
+	<axis xyz="0 1 0"/>
+    <dynamics damping="0.7"/>
+  </joint>
+  <link name="wrist_link1">
+    <collision>
+		<origin xyz="0 0 ${height_w1/2}" rpy="0 0 0"/>
+      <geometry>
+		  <!--box size="${width_w1} ${width_w1*4} ${height_w1}"/-->
+     	<mesh filename="${model_wrist1}" scale="0 0 0" />
+      </geometry>
+    </collision>
+    <visual>
+		<origin xyz="0 0 ${height_w1/2}" rpy="0 0 0"/>
+      <geometry>
+		<!--box size="${width_w1} ${width_w1*4} ${height_w1}"/-->
+		<mesh filename="${model_wrist1}" scale="${model_scale}" />
+      </geometry>
+      <material name="orange"/>
+    </visual>
+    <inertial>
+		<origin xyz="0 0 ${height_w1/2}" rpy="0 0 0"/>
+      <mass value="${mass_w1}"/>
+      <inertia
+	  ixx="${mass_w1 / 1.0  * (width_w1*width_w1 + height_w1*height_w1)}" ixy="0.0" ixz="0.0"
+	  iyy="${mass_w1 / 1.0  * (height_w1*height_w1 + width_w1*width_w1)}" iyz="0.0"
+	  izz="${mass_w1 / 1.0  * (width_w1*width_w1 + width_w1*width_w1)}"/>
+    </inertial>
+  </link>
+  <joint name="wrist_joint2" type="continuous">
+    <parent link="wrist_link1"/>
+    <child link="wrist_link2"/>
+		<origin xyz="-0.01 0 ${height_w2-0.001}" rpy="0 0 0"/>
+	<axis xyz="0 1 0"/>
+    <dynamics damping="0.7"/>
+  </joint>
+  <link name="wrist_link2">
+    <collision>
+		<origin xyz="0 0 ${height_w2/2}" rpy="0 0 0"/>
+      <geometry>
+		  <!--box size="${width_w2} ${width_w2*4} ${height_w2}"/-->
+     	<mesh filename="${model_wrist2}" scale="0 0 0" />
+      </geometry>
+    </collision>
+    <visual>
+		<origin xyz="0 0 ${height_w2/2}" rpy="0 0 0"/>
+      <geometry>
+		<!--box size="${width_w2} ${width_w2*4} ${height_w2}"/-->
+		<mesh filename="${model_wrist2}" scale="${model_scale}" />
+      </geometry>
+      <material name="orange"/>
+    </visual>
+    <inertial>
+		<origin xyz="0 0 ${height_w2/2}" rpy="0 0 0"/>
+      <mass value="${mass_w2}"/>
+      <inertia
+	  ixx="${mass_w2 / 1.0  * (width_w2*width_w2 + height_w2*height_w2)}" ixy="0.0" ixz="0.0"
+	  iyy="${mass_w2 / 1.0  * (height_w2*height_w2 + width_w2*width_w2)}" iyz="0.0"
+	  izz="${mass_w2 / 1.0  * (width_w2*width_w2 + width_w2*width_w2)}"/>
+    </inertial>
+  </link>
+  <joint name="wrist_connector" type="fixed">
+	  <parent link="wrist_link2"/>
+	  <child link="palm"/>
+	  <origin xyz="-0.009 0.013 ${height_w2+0.013}" rpy="0 0 0"/>
+  </joint>
+<!--**************** Palm ********************-->
+  <link name="palm">
+    <collision>
+		<origin xyz="0 0 ${height_p/2}" rpy="0 0 0"/>
+      <geometry>
+		  <!--box size="${width/2} ${width_p} ${height_p}"/-->
+		<mesh filename="${model_palm}" scale="${model_scale}" />
+      </geometry>
+    </collision>
+    <visual>
+		<origin xyz="0 0 ${height_p/2}" rpy="0 0 0"/>
+      <geometry>
+		  <!--box size="${width/2} ${width_p} ${height_p}"/-->
+		<mesh filename="${model_palm}" scale="${model_scale}" />
+      </geometry>
+      <material name="orange"/>
+    </visual>
+    <inertial>
+		<origin xyz="0 0 ${height_p/2}" rpy="0 0 0"/>
+      <mass value="${mass}"/>
+      <inertia
+	  ixx="${mass*3 / 1.0  * (width_p*width_p + height_p*height_p)}" ixy="0.0" ixz="0.0"
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